Commit message: Kinova Gen3 7DoF added to the model.

File: urdf/P3Bot.urdf.xacro (robot description, xacro)
@@ -11,5 +11,5 @@
   <xacro:include filename="$(find p3bot_description)/urdf/base.xacro"/>
   <xacro:include filename="$(find p3bot_description)/urdf/wheels.xacro"/>
-  <!--  ||||||||TODO||||||||   <xacro:include filename="$(find p3bot_description)/urdf/kinova_arm.xacro"/> -->
+  <xacro:include filename="$(find p3bot_description)/urdf/GEN3_URDF_V12.xacro"/>
   <xacro:include filename="$(find p3bot_description)/urdf/sensors.xacro"/>
   <!-- ====== BASE ====== -->
@@ -17,16 +17,25 @@
   <!-- ====== WHEELS ====== -->
   <xacro:p3bot_wheels parent="base_link"/>
-  <!-- ====== ARMS ====== ||||||||TODO||||||||
+  <!-- ====== ARMS ====== |-->
   <xacro:if value="$(arg left_arm)">
-    <xacro:kinova_arm prefix="left_" parent="base_link"
-      xyz="0.002 0.055 1.052"
-      rpy="-2.010005 0 0"/>
+    <link name="left_arm_mount"/>
+    <joint name="left_arm_mount_joint" type="fixed">
+      <parent link="base_link"/>
+      <child link="left_arm_mount"/>
+      <origin xyz="0.002 0.055 1.052"
+              rpy="1.13159 0 0"/>
+    </joint>
+    <xacro:GEN3_URDF_V12 prefix="left_" parent="left_arm_mount"/>
   </xacro:if>
   <xacro:if value="$(arg right_arm)">
-    <xacro:kinova_arm prefix="right_" parent="base_link"
-      xyz="0.01 -0.051761 1.04883"
-      rpy="2.01001 0 0"/>
+    <link name="right_arm_mount"/>
+    <joint name="right_arm_mount_joint" type="fixed">
+      <parent link="base_link"/>
+      <child link="right_arm_mount"/>
+      <origin xyz="0.01 -0.051761 1.04883"
+              rpy="-1.13159 0 0"/>
+    </joint>
+    <xacro:GEN3_URDF_V12 prefix="right_" parent="right_arm_mount"/>
   </xacro:if>
-  -->
   <!-- ====== SENSORS ====== -->
   <xacro:p3bot_sensors parent="base_link"/>

File: urdf/sensors.xacro (robot description, xacro)
@@ -6,5 +6,5 @@
       <parent link="${parent}"/>
       <child link="zed_link"/>
-      <origin xyz="0.01 0 1.32" rpy="-1.570796 0 -1.570796"/>
+      <origin xyz="0.07 0 1.1"/>
     </joint>
     <link name="imu_link"/>
@@ -14,4 +14,16 @@
       <origin xyz="0 0 0"/>
     </joint>
+    <link name="helios_link"/>
+    <joint name="base_to_helios" type="fixed">
+      <parent link="${parent}"/>
+      <child link="helios_link"/>
+      <origin xyz="-0.05 0 1.24"/>
+    </joint>
+    <link name="camera_360_link"/>
+    <joint name="base_to_camera_360" type="fixed">
+      <parent link="${parent}"/>
+      <child link="camera_360_link"/>
+      <origin xyz="-0.05 0 1.42"/>
+    </joint>
   </xacro:macro>
 </robot>
